File: updatedMinibadge/updatedMinibadge.kicad_sch (KiCad schematic)
At the start: 1 part

Commit message: Added logo
Changed lines of the file:
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@@
 			)
-		)
-		(pin "11"
-		)
-		(pin "6"
 		)
 		(pin "1"
@@
 		(pin "8"
 		)
-		(pin "3"
-		)
 		(pin "2"
 		)
 		(pin "13"
 		)
-		(pin "12"
-		)
-		(pin "5"
-		)
-		(pin "4"
-		)
 		(pin "7"
