File: updatedMinibadge/updatedMinibadge.kicad_pcb (KiCad board)
At the start: 2 copper layers, 1 part

Commit message: updated footprints
Parts:
- removed the REF** at (123.8, 69.7)
- added REF**: MiniBadge_Full, MiniBadge:MiniBadge_Full, F.Cu at (139.2, 87.1)
Other:
- board outline added: 20 x 20 mm
